File: arudino-clone.kicad_pcb (KiCad board)
At the start: 2 copper layers, 68.8 x 53.6 mm, 39 parts, among them J101 Barrel_Jack, J102 Conn_01x08, J103 Conn_01x08, J104 Conn_01x06, J105 Conn_01x10, J106 AVR-ISP-6, J201 USB_C_Receptacle_USB2.0, SW101 SW_SPST, U101 LM317, U102 AMS1117-3.3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

Commit message: updated caps and power regulator
Parts:
- removed R103: 3K74, Capacitor_SMD:C_0805_2012Metric
- removed R104: 330, Resistor_SMD:R_0603_1608Metric
- added C110: 100nF, Capacitor_SMD:C_0603_1608Metric, F.Cu at (137.2, 85.6)
- added C111: 100nF, Capacitor_SMD:C_0603_1608Metric, F.Cu at (138.4, 86.9)
- added C112: 100nF, Capacitor_SMD:C_0603_1608Metric, F.Cu at (119.1, 95.8)
- added C202: 100nF, Capacitor_SMD:C_0603_1608Metric, F.Cu at (110.0, 76.5)
- C101, C103: value 100nF -> 10uF; footprint Capacitor_SMD:C_0603_1608Metric -> Capacitor_SMD:C_0805_2012Metric
- C108: value 1uF -> 10uF; footprint Capacitor_SMD:C_0603_1608Metric -> Capacitor_SMD:C_0805_2012Metric
- C201: value 22uF -> 10uF
- J102: value Conn_01x08 -> Conn_01x06; footprint Connector_PinSocket_2.54mm:PinSocket_1x08_P2.54mm_Vertical -> Connector_PinSocket_2.54mm:PinSocket_1x06_P2.54mm_Vertical
- J104: value Conn_01x06 -> Conn_01x10; footprint Connector_PinSocket_2.54mm:PinSocket_1x06_P2.54mm_Vertical -> Connector_PinSocket_2.54mm:PinSocket_1x10_P2.54mm_Vertical
- J105: value Conn_01x10 -> Conn_01x08; footprint Connector_PinSocket_2.54mm:PinSocket_1x10_P2.54mm_Vertical -> Connector_PinSocket_2.54mm:PinSocket_1x08_P2.54mm_Vertical
- R102: value 10K -> 330
- U101: value LM317 -> AMS1117-5.0
- moved J105 50.2 mm to (114.3, 115.6), turned to 90 degrees
- moved J104 49.1 mm to (128.0, 67.3), turned to -90 degrees
- moved C101 25.8 mm to (104.4, 110.0), turned to 90 degrees
- moved C102 23.0 mm to (105.7, 106.9), turned to 180 degrees
- moved J102 22.9 mm to (137.2, 115.6)
- moved FB102 18.8 mm to (120.7, 94.5), turned to 135 degrees
- moved C107 18.5 mm to (123.2, 96.8), turned to -45 degrees
- moved C103 15.4 mm to (108.3, 104.4)
- moved U101 11.4 mm to (102.6, 98.6), turned to 90 degrees
- moved C108 10.9 mm to (113.0, 89.9)
- moved R102 8.83 mm to (104.8, 89.9)
- moved F101 5.84 mm to (101.3, 109.7), turned to -90 degrees
- moved FB101 4.13 mm to (106.9, 110.0), turned to 90 degrees
- moved C104 2.71 mm to (101.6, 104.4), turned to 180 degrees
- moved U102 2.05 mm to (93.5, 92.5), turned to 90 degrees
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Connections:
- C101 pad 1: +5V -> Net-(C101-Pad1)
- C102 pad 1: +5V -> VBUS
- C103 pad 1: /AREF -> VBUS
- C104 pad 1: Net-(C104-Pad1) -> +5V
- C107 pad 1: VBUS -> /AREF
- F101 pad 2: Net-(C104-Pad1) -> Net-(C101-Pad1)
- FB101 pad 1: Net-(C104-Pad1) -> Net-(C101-Pad1)
- J102 pad 1: unconnected-(J102-Pin_1-Pad1) -> /PC0
- J102 pad 2: +5V -> /PC1
- J102 pad 3: /~{RESET} -> /PC2
- J102 pad 4: +3V3 -> /PC3
- J102 pad 5: +5V -> /PC4
- J102 pad 6: GND -> /PC5
- J104 pad 1: /PC0 -> /PB0
- J104 pad 2: /PC1 -> /PB1
- J104 pad 3: /PC2 -> /PB2
- J104 pad 4: /PC3 -> /PB3
- J104 pad 5: /PC4 -> /PB4
- J104 pad 6: /PC5 -> /PB5
- J105 pad 1: /PB0 -> unconnected-(J105-Pin_1-Pad1)
- J105 pad 2: /PB1 -> +5V
- J105 pad 3: /PB2 -> /~{RESET}
- J105 pad 4: /PB3 -> +3V3
- J105 pad 5: /PB4 -> +5V
- J105 pad 6: /PB5 -> GND
- J105 pad 8: /AREF -> unconnected-(J105-Pin_8-Pad8)
- R102 pad 1: +5V -> /~{RESET}
- R102 pad 2: Net-(U101-ADJ) -> Net-(SW101-A)
- U101 pad 1: Net-(U101-ADJ) -> GND
